File: KiCad/diy_tdr/diy_tdr.sch (KiCad schematic (older format))
At the start: 30 parts, among them J1 DUT, J2 Scope, J3 Trig, SW1 SW_SPDT, U1 74HC14, sw1 A10503RNCQ, sw2 A10503RNCQ

Commit message: Foot Prints Added
Parts:
- BT1: footprint (none) -> Symacy:2479
- SW1: footprint (none) -> Symacy:M2012LL1W03
- sw1, sw2: footprint (none) -> Symacy:A10405RNCQE; symbol Switch:A10503RNCQ -> diy_tdr-rescue:A10503RNCQ-Switch
Changed lines of the file:
@@
 $EndComp
 $Comp
-L Switch:A10503RNCQ sw2
+L diy_tdr-rescue:A10503RNCQ-Switch sw2
 U 1 1 61F34E21
 P 7850 3850
 F 0 "sw2" V 8228 3271 50  0000 L CNN
 F 1 "A10503RNCQ" V 8350 3050 50  0000 L CNN
-F 2 "" H 7650 3550 50  0001 C CNN
+F 2 "Symacy:A10405RNCQE" H 7650 3550 50  0001 C CNN
 F 3 "" H 7650 3550 50  0001 C CNN
 	1    7850 3850
@@
 $EndComp
 $Comp
-L Switch:A10503RNCQ sw1
+L diy_tdr-rescue:A10503RNCQ-Switch sw1
 U 1 1 61F372C4
 P 4050 3900
 F 0 "sw1" H 4150 3500 50  0000 L CNN
 F 1 "A10503RNCQ" H 3450 3500 50  0000 L CNN
-F 2 "" H 3850 3600 50  0001 C CNN
+F 2 "Symacy:A10405RNCQE" H 3850 3600 50  0001 C CNN
 F 3 "" H 3850 3600 50  0001 C CNN
 	1    4050 3900
@@
 F 0 "BT1" V 1355 6150 50  0000 C CNN
 F 1 "Battery" V 1446 6150 50  0000 C CNN
-F 2 "" V 1600 6210 50  0001 C CNN
+F 2 "Symacy:2479" V 1600 6210 50  0001 C CNN
 F 3 "~" V 1600 6210 50  0001 C CNN
 	1    1600 6150
@@
 F 0 "SW1" H 2100 6435 50  0000 C CNN
 F 1 "SW_SPDT" H 2100 6344 50  0000 C CNN
-F 2 "" H 2100 6150 50  0001 C CNN
+F 2 "Symacy:M2012LL1W03" H 2100 6150 50  0001 C CNN
 F 3 "~" H 2100 6150 50  0001 C CNN
 	1    2100 6150

Commit message: finished layout
Parts:
- removed sw1, sw2: A10503RNCQ, Symacy:A10405RNCQE, symbol diy_tdr-rescue:A10503RNCQ-Switch
- added RV1: R_POT_TRIM_US, Potentiometer_THT:Potentiometer_Runtron_RM-065_Vertical, symbol Device:R_POT_TRIM_US
- added S1, S2: A10303RNCB, A10405RNCQE, symbol SamacSys_Parts:A10503RNCQ
- BT1: footprint Symacy:2479 -> SamacSys_Parts:2479
- D2: footprint (none) -> LED_THT:LED_D3.0mm
- J1, J2, J3: footprint Connector_Coaxial:BNC_Amphenol_B6252HB-NPP3G-50_Horizontal -> SamacSys_Parts:731375003
- SW1: footprint Symacy:M2012LL1W03 -> SamacSys_Parts:M2012LL1W03
Connections:
- net at D1.2 (A), R1.2, U1.1: now also RV1.3, S2.A1 (COM)
- net at R1.1, R2.1, U1.11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: now also RV1.1, RV1.2
- net at C1.1: now also S2.1 (NO_0)
- net at J1.1 (In), J2.1 (In): now also S1.A1 (COM)
- net at R10.2, R11.2, R12.2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: now also S1.1 (NO_0), S1.2 (NO_1)
- net at R11.1: now also S1.3 (NO_2)
- net at R10.1: now also S1.4 (NO_3), S1.5 (NO_4)
- net at C2.1: now also S2.2 (NO_1)
- net at C3.1: now also S2.3 (NO_2)
- net at C4.1: now also S2.4 (NO_3)
- net at C5.1: now also S2.5 (NO_4)
- net at SW1.1 (A): now also R3.2
- net at SW1.3 (C): no longer R3.2
- new net: S2.10 (NO_CONNECTION_5), S2.11 (NO_CONNECTION_6), S2.12 (NO_CONNECTION_7), S2.6 (NO_CONNECTION_1), S2.7 (NO_CONNECTION_2), S2.8 (NO_CONNECTION_3), S2.9 (NO_CONNECTION_4)
- new net: S1.10 (NO_CONNECTION_5), S1.11 (NO_CONNECTION_6), S1.12 (NO_CONNECTION_7), S1.6 (NO_CONNECTION_1), S1.7 (NO_CONNECTION_2), S1.8 (NO_CONNECTION_3), S1.9 (NO_CONNECTION_4)
Other:
- moved on the sheet: C1, C2, C3, C4, C5, J1, J2, J3
